File: boards/Digital Synth/MIDI.sch (KiCad schematic (older format))
At the start: 11 parts, among them J3 DIN-5, J4 DIN-5, U4 6N138, U5 74LS14

Commit message: progress on layout for DAC and MIDI
Parts:
- removed U5: 74LS14, symbol 74xx:74LS14
- added U2: SN74LVC2G14, Package_TO_SOT_SMD:SOT-23-6_Handsoldering, symbol 74xx:SN74LVC2G14
- C25: footprint (none) -> Capacitor_SMD:C_0603_1608Metric_Pad1.05x0.95mm_HandSolder
- D30: footprint (none) -> Diode_SMD:D_0805_2012Metric_Pad1.15x1.40mm_HandSolder
- J3, J4: footprint (none) -> Connector_Audio_Ext:MIDI_DIN5
- R5, R6, R7, R8, R9: footprint (none) -> Resistor_SMD:R_0805_2012Metric_Pad1.15x1.40mm_HandSolder
- U4: footprint (none) -> Package_DIP:SMDIP-8_W7.62mm
Changed lines of the file:
@@
 F 0 "U4" H 4050 4617 50  0000 C CNN
 F 1 "6N138" H 4050 4526 50  0000 C CNN
-F 2 "" H 4340 3850 50  0001 C CNN
+F 2 "Package_DIP:SMDIP-8_W7.62mm" H 4340 3850 50  0001 C CNN
 F 3 "http://www.onsemi.com/pub/Collateral/HCPL2731-D.pdf" H 4340 3850 50  0001 C CNN
 	1    4050 4150
@@
 F 0 "R7" H 4984 4071 50  0000 L CNN
 F 1 "1k" H 4984 3980 50  0000 L CNN
-F 2 "" H 4925 4025 50  0001 C CNN
+F 2 "Resistor_SMD:R_0805_2012Metric_Pad1.15x1.40mm_HandSolder" H 4925 4025 50  0001 C CNN
 F 3 "~" H 4925 4025 50  0001 C CNN
 	1    4925 4025
@@
 F 0 "J3" V 2854 3920 50  0000 R CNN
 F 1 "DIN-5" V 2945 3920 50  0000 R CNN
-F 2 "" H 2900 4150 50  0001 C CNN
+F 2 "Connector_Audio_Ext:MIDI_DIN5" H 2900 4150 50  0001 C CNN
 F 3 "http://www.mouser.com/ds/2/18/40_c091_abd_e-75918.pdf" H 2900 4150 50  0001 C CNN
 	1    2900 4150
@@
 F 0 "R6" H 4809 4471 50  0000 L CNN
 F 1 "10k" H 4809 4380 50  0000 L CNN
-F 2 "" H 4750 4425 50  0001 C CNN
+F 2 "Resistor_SMD:R_0805_2012Metric_Pad1.15x1.40mm_HandSolder" H 4750 4425 50  0001 C CNN
 F 3 "~" H 4750 4425 50  0001 C CNN
 	1    4750 4425
@@
 F 0 "R5" V 3054 3850 50  0000 C CNN
 F 1 "220" V 3145 3850 50  0000 C CNN
-F 2 "" H 3250 3850 50  0001 C CNN
+F 2 "Resistor_SMD:R_0805_2012Metric_Pad1.15x1.40mm_HandSolder" H 3250 3850 50  0001 C CNN
 F 3 "~" H 3250 3850 50  0001 C CNN
 	1    3250 3850
@@
 F 0 "D30" V 3525 3925 50  0000 L CNN
 F 1 "1N4148" V 3675 3800 50  0000 L CNN
-F 2 "" V 3575 4125 50  0001 C CNN
+F 2 "Diode_SMD:D_0805_2012Metric_Pad1.15x1.40mm_HandSolder" V 3575 4125 50  0001 C CNN
 F 3 "~" V 3575 4125 50  0001 C CNN
 	1    3575 4125
@@
 F 0 "C25" V 4425 3850 50  0000 C CNN
 F 1 "0.1uF" V 4500 3850 50  0000 C CNN
-F 2 "" H 4625 3800 50  0001 C CNN
+F 2 "Capacitor_SMD:C_0603_1608Metric_Pad1.05x0.95mm_HandSolder" H 4625 3800 50  0001 C CNN
 F 3 "~" H 4625 3800 50  0001 C CNN
 	1    4625 3800
@@
 Wire Notes Line
 	2400 4975 5525 4975
-$Comp
-L 74xx:74LS14 U5
-U 1 1 621D0DE5
-P 6950 4575
-F 0 "U5" H 6950 4892 50  0000 C CNN
-F 1 "74LS14" H 6950 4801 50  0000 C CNN
-F 2 "" H 6950 4575 50  0001 C CNN
-F 3 "http://www.ti.com/lit/gpn/sn74LS14" H 6950 4575 50  0001 C CNN
-	1    6950 4575
-	1    0    0    -1
-$EndComp
-$Comp
-L 74xx:74LS14 U5
-U 2 1 621D3679
-P 7550 4575
-F 0 "U5" H 7550 4892 50  0000 C CNN
-F 1 "74LS14" H 7550 4801 50  0000 C CNN
-F 2 "" H 7550 4575 50  0001 C CNN
-F 3 "http://www.ti.com/lit/gpn/sn74LS14" H 7550 4575 50  0001 C CNN
-	2    7550 4575
-	1    0    0    -1
-$EndComp
 Text GLabel 6500 4575 0    50   Input ~ 0
 TXD
@@
 F 0 "R8" V 7829 4575 50  0000 C CNN
 F 1 "220" V 7920 4575 50  0000 C CNN
-F 2 "" H 8025 4575 50  0001 C CNN
+F 2 "Resistor_SMD:R_0805_2012Metric_Pad1.15x1.40mm_HandSolder" H 8025 4575 50  0001 C CNN
 F 3 "~" H 8025 4575 50  0001 C CNN
 	1    8025 4575
@@
 F 0 "J4" V 8700 3850 50  0000 C CNN
 F 1 "DIN-5" V 8800 3850 50  0000 C CNN
-F 2 "" H 8650 4175 50  0001 C CNN
+F 2 "Connector_Audio_Ext:MIDI_DIN5" H 8650 4175 50  0001 C CNN
 F 3 "http://www.mouser.com/ds/2/18/40_c091_abd_e-75918.pdf" H 8650 4175 50  0001 C CNN
 	1    8650 4175
@@
 F 0 "R9" H 8609 3746 50  0000 L CNN
 F 1 "220" H 8609 3655 50  0000 L CNN
-F 2 "" H 8550 3700 50  0001 C CNN
+F 2 "Resistor_SMD:R_0805_2012Metric_Pad1.15x1.40mm_HandSolder" H 8550 3700 50  0001 C CNN
 F 3 "~" H 8550 3700 50  0001 C CNN
 	1    8550 3700
@@
 $EndComp
 $Comp
-L 74xx:74LS14 U5
-U 7 1 62245149
-P 7350 3800
-F 0 "U5" V 7675 3875 50  0000 L CNN
-F 1 "74LS14" V 7600 3750 50  0000 L CNN
-F 2 "" H 7350 3800 50  0001 C CNN
-F 3 "http://www.ti.com/lit/gpn/sn74LS14" H 7350 3800 50  0001 C CNN
-	7    7350 3800
-	0    -1   -1   0
-$EndComp
-$Comp
 L power:+5V #PWR034
 U 1 1 6224948F
-P 6825 3775
-F 0 "#PWR034" H 6825 3625 50  0001 C CNN
-F 1 "+5V" H 6840 3948 50  0000 C CNN
-F 2 "" H 6825 3775 50  0001 C CNN
-F 3 "" H 6825 3775 50  0001 C CNN
-	1    6825 3775
-	1    0    0    -1
-$EndComp
-Wire Wire Line
-	6825 3800 6850 3800
+P 6950 3750
+F 0 "#PWR034" H 6950 3600 50  0001 C CNN
+F 1 "+5V" H 6965 3923 50  0000 C CNN
+F 2 "" H 6950 3750 50  0001 C CNN
+F 3 "" H 6950 3750 50  0001 C CNN
+	1    6950 3750
+	1    0    0    -1
+$EndComp
+Wire Wire Line
+	6950 3775 6975 3775
 $Comp
 L power:GND #PWR035
 U 1 1 6224AD25
-P 7875 3825
-F 0 "#PWR035" H 7875 3575 50  0001 C CNN
-F 1 "GND" H 7880 3652 50  0000 C CNN
-F 2 "" H 7875 3825 50  0001 C CNN
-F 3 "" H 7875 3825 50  0001 C CNN
-	1    7875 3825
-	1    0    0    -1
-$EndComp
-Wire Wire Line
-	7875 3800 7850 3800
-Wire Wire Line
-	6825 3775 6825 3800
-Wire Wire Line
-	7875 3800 7875 3825
+P 7700 3800
+F 0 "#PWR035" H 7700 3550 50  0001 C CNN
+F 1 "GND" H 7705 3627 50  0000 C CNN
+F 2 "" H 7700 3800 50  0001 C CNN
+F 3 "" H 7700 3800 50  0001 C CNN
+	1    7700 3800
+	1    0    0    -1
+$EndComp
+Wire Wire Line
+	7700 3775 7675 3775
+Wire Wire Line
+	6950 3750 6950 3775
+Wire Wire Line
+	7700 3775 7700 3800
+$Comp
+L 74xx:SN74LVC2G14 U2
+U 1 1 61FDAC18
+P 6900 4575
+F 0 "U2" H 6950 4892 50  0000 C CNN
+F 1 "SN74LVC2G14" H 6950 4801 50  0000 C CNN
+F 2 "Package_TO_SOT_SMD:SOT-23-6_Handsoldering" H 6900 4775 50  0001 C CNN
+F 3 "" H 6900 4775 50  0001 C CNN
+	1    6900 4575
+	1    0    0    -1
+$EndComp
+$Comp
+L 74xx:SN74LVC2G14 U2
+U 2 1 61FE5EE1
+P 7325 3775
+F 0 "U2" H 7325 3500 50  0000 C CNN
+F 1 "SN74LVC2G14" H 7300 3575 50  0000 C CNN
+F 2 "Package_TO_SOT_SMD:SOT-23-6_Handsoldering" H 7325 3975 50  0001 C CNN
+F 3 "" H 7325 3975 50  0001 C CNN
+	2    7325 3775
+	-1   0    0    1
+$EndComp
+$Comp
+L 74xx:SN74LVC2G14 U2
+U 3 1 61FE6C72
+P 7500 4575
+F 0 "U2" H 7550 4892 50  0000 C CNN
+F 1 "SN74LVC2G14" H 7550 4801 50  0000 C CNN
+F 2 "Package_TO_SOT_SMD:SOT-23-6_Handsoldering" H 7500 4775 50  0001 C CNN
+F 3 "" H 7500 4775 50  0001 C CNN
+	3    7500 4575
+	1    0    0    -1
+$EndComp
 $EndSCHEMATC

Commit message: laid out keyboard
Parts:
- removed C25: 0.1uF, Capacitor_SMD:C_0603_1608Metric_Pad1.05x0.95mm_HandSolder, symbol device:C_Small
- removed D30: 1N4148, Diode_SMD:D_0805_2012Metric_Pad1.15x1.40mm_HandSolder, symbol device:D_Small
- removed J3, J4: DIN-5, Connector_Audio_Ext:MIDI_DIN5, symbol Connector:DIN-5_180degree
- removed R5, R8, R9: 220, Resistor_SMD:R_0805_2012Metric_Pad1.15x1.40mm_HandSolder, symbol device:R_Small
- removed R6: 10k, Resistor_SMD:R_0805_2012Metric_Pad1.15x1.40mm_HandSolder, symbol device:R_Small
- removed R7: 1k, Resistor_SMD:R_0805_2012Metric_Pad1.15x1.40mm_HandSolder, symbol device:R_Small
- removed U2: SN74LVC2G14, Package_TO_SOT_SMD:SOT-23-6_Handsoldering, symbol 74xx:SN74LVC2G14
- removed U4: 6N138, Package_DIP:SMDIP-8_W7.62mm, symbol Isolator:6N138
Connections:
- no-connect marks 5 -> 0
Other:
- note removed: "MIDI In"
- note removed: "MIDI Out"
